File: _saved_rpi_ext.sch (KiCad schematic (older format))
At the start: 100 parts, among them J10 CONN_01X22, J11 CONN_01X22, J12 CONN_01X22, J13 HDMI, J14 USB_HOST, J15 USB_SLAVE, J16 Micro_SD_Card, J2 USB_POWER, J3 CONN_02X03, J4 CONN_01X03, J5 CONN_02X30, J6 CONN_02X30, J7 CONN_01X08, J9 CONN_01X22, Q1 DMG1012T, Q2 DMG1012T, Q4 DMG1012T, Q5 DMG1012T, U1 PAM2306AYPKE, U2 AP7115-25SEG, U3 AP2331W, U4 ESD5384, U5 FSUSB42UMX

Commit message: SCH DONE
Parts:
- C1, C10, C11, C12, C13, C14, C15, C16, C17, C19, C2, C20, C21, C22, C23, C24, C3, C4, C5, C6, C7, C8, C9: footprint (none) -> Capacitors_SMD:C_0603_HandSoldering
- D1, D2: footprint (none) -> LEDs:LED_0606
- J3: value CONN_02X03 -> GPIO VOLTAGE SELECT
- R1, R10, R12, R13, R14, R15, R16, R17, R18, R19, R2, R20, R21, R22, R23, R24, R25, R26, R27, R28, R29, R3, R30, R31, R4, R5, R6, R7, R8, R9: footprint (none) -> Resistors_SMD:R_0603_HandSoldering
- gave numbers to parts that had none: 2
